Commit message: added primitive gazebo capabilities

File: sec_test_dev_ws/install/sec_description/share/sec_description/description/sec_description_final.urdf.xacro (robot description, xacro)
@@ -8,5 +8,6 @@
 	<!-- These make use of xacro's mathematical functionality -->
 	<!-- Base Footprint -->
-	<link name="base_link"/>
+	<link name="base_link">
+    </link>
 	<!-- Robot Base -->
 	<link name="chassis">
@@ -37,5 +38,5 @@
 		<origin rpy="0 0 0" xyz="0.0 0.0 0.05"/>
 	</joint>
-	<link name="drivewhl_l_link">
+	<link name="b_l_wheel_link">
 		<visual>
 			<origin rpy="1.5707963267948966 0 0" xyz="0 0 0"/>
@@ -59,11 +60,14 @@
 		</inertial>
 	</link>
-	<joint name="drivewhl_lbase_joint" type="continuous">
+	<joint name="b_l_wheel_joint" type="continuous">
 		<parent link="chassis"/>
-		<child link="drivewhl_l_link"/>
+		<child link="b_l_wheel_link"/>
 		<origin rpy="0 0 0" xyz="-0.125 0.3 0.03"/>
 		<axis xyz="0 1 0"/>
 	</joint>
-	<link name="drivewhl_r_link">
+	<gazebo reference="b_l_wheel_link">
+		<material>Gazebo/Blue</material>
+	</gazebo>
+	<link name="b_r_wheel_link">
 		<visual>
 			<origin rpy="1.5707963267948966 0 0" xyz="0 0 0"/>
@@ -87,11 +91,14 @@
 		</inertial>
 	</link>
-	<joint name="drivewhl_rbase_joint" type="continuous">
+	<joint name="b_r_wheel_joint" type="continuous">
 		<parent link="chassis"/>
-		<child link="drivewhl_r_link"/>
+		<child link="b_r_wheel_link"/>
 		<origin rpy="0 0 0" xyz="-0.125 -0.3 0.03"/>
 		<axis xyz="0 1 0"/>
 	</joint>
-	<link name="frontwhl_l_link">
+	<gazebo reference="b_r_wheel_link">
+		<material>Gazebo/Blue</material>
+	</gazebo>
+	<link name="f_l_wheel_link">
 		<visual>
 			<origin rpy="1.5707963267948966 0 0" xyz="0 0 0"/>
@@ -115,11 +122,14 @@
 		</inertial>
 	</link>
-	<joint name="frontwhl_lbase_joint" type="continuous">
+	<joint name="f_l_wheel_joint" type="continuous">
 		<parent link="chassis"/>
-		<child link="frontwhl_l_link"/>
+		<child link="f_l_wheel_link"/>
 		<origin rpy="0 0 0" xyz="0.125 0.3 0.03"/>
 		<axis xyz="0 1 0"/>
 	</joint>
-	<link name="frontwhl_r_link">
+	<gazebo reference="f_l_wheel_link">
+		<material>Gazebo/Blue</material>
+	</gazebo>
+	<link name="f_r_wheel_link">
 		<visual>
 			<origin rpy="1.5707963267948966 0 0" xyz="0 0 0"/>
@@ -143,9 +153,38 @@
 		</inertial>
 	</link>
-	<joint name="frontwhl_rbase_joint" type="continuous">
+	<joint name="f_r_wheel_joint" type="continuous">
 		<parent link="chassis"/>
-		<child link="frontwhl_r_link"/>
+		<child link="f_r_wheel_link"/>
 		<origin rpy="0 0 0" xyz="0.125 -0.3 0.03"/>
 		<axis xyz="0 1 0"/>
 	</joint>
+	<gazebo reference="f_r_wheel_link">
+		<material>Gazebo/Blue</material>
+	</gazebo>
+	<gazebo>
+		<plugin filename="libgazebo_ros_diff_drive.so" name="four_wheeled_robot_diff_drive">
+			<!-- Number of wheel pairs -->
+			<num_wheel_pairs>2</num_wheel_pairs>
+			<!-- wheels0 -->
+			<left_joint>f_l_wheel_joint</left_joint>
+			<right_joint>f_r_wheel_joint</right_joint>
+			<!-- wheels1-->
+			<left_joint>b_l_wheel_joint</left_joint>
+			<right_joint>b_r_wheel_joint</right_joint>
+			<!-- kinematics -->
+			<wheel_separation>&quot;0.5&quot;</wheel_separation>
+			<wheel_separation>&quot;0.5&quot;</wheel_separation>
+			<wheel_diameter>0.2</wheel_diameter>
+			<wheel_diameter>0.2</wheel_diameter>
+			<!-- limits -->
+			<max_wheel_torque>200</max_wheel_torque>
+			<max_wheel_acceleration>10.0</max_wheel_acceleration>
+			<!-- output -->
+			<publish_odom>true</publish_odom>
+			<publish_odom_tf>true</publish_odom_tf>
+			<publish_wheel_tf>true</publish_wheel_tf>
+			<odometry_frame>odom</odometry_frame>
+			<robot_base_frame>chassis</robot_base_frame>
+		</plugin>
+	</gazebo>
 </robot>

File: sec_test_dev_ws/src/sec_description/description/gazebo_control.xacro (robot description, xacro)
@@ -2,4 +2,28 @@
 <robot xmlns:xacro="http://www.ros.org/wiki/xacro">
     <gazebo>
+        <plugin name="four_wheeled_robot_diff_drive" filename="libgazebo_ros_diff_drive.so">
+            <!-- Number of wheel pairs -->
+            <num_wheel_pairs>2</num_wheel_pairs>
+            <!-- wheels0 -->
+            <left_joint>f_l_wheel_joint</left_joint>
+            <right_joint>f_r_wheel_joint</right_joint>
+            <!-- wheels1-->
+            <left_joint>b_l_wheel_joint</left_joint>
+            <right_joint>b_r_wheel_joint</right_joint>
+            <!-- kinematics -->
+            <wheel_separation>"${chassis_width}"</wheel_separation>
+            <wheel_separation>"${chassis_width}"</wheel_separation>
+            <wheel_diameter>${wheel_radius*2}</wheel_diameter>
+            <wheel_diameter>${wheel_radius*2}</wheel_diameter>
+            <!-- limits -->
+            <max_wheel_torque>200</max_wheel_torque>
+            <max_wheel_acceleration>10.0</max_wheel_acceleration>
+            <!-- output -->
+            <publish_odom>true</publish_odom>
+            <publish_odom_tf>true</publish_odom_tf>
+            <publish_wheel_tf>true</publish_wheel_tf>
+            <odometry_frame>odom</odometry_frame>
+            <robot_base_frame>chassis</robot_base_frame>
+        </plugin>
     </gazebo>
 </robot>

File: sec_test_dev_ws/src/sec_description/description/inertial_macros.xacro (robot description, xacro)
@@ -6,8 +6,8 @@
         <inertial>
             <xacro:insert_block name="origin"/>
-            <mass value="${mass}" />
+            <mass value="${mass}"/>
             <inertia ixx="${(2/5) * mass * (radius*radius)}" ixy="0.0" ixz="0.0"
-                    iyy="${(2/5) * mass * (radius*radius)}" iyz="0.0"
-                    izz="${(2/5) * mass * (radius*radius)}" />
+                     iyy="${(2/5) * mass * (radius*radius)}" iyz="0.0"
+                     izz="${(2/5) * mass * (radius*radius)}"/>
         </inertial>
     </xacro:macro>
@@ -15,8 +15,8 @@
         <inertial>
             <xacro:insert_block name="origin"/>
-            <mass value="${mass}" />
+            <mass value="${mass}"/>
             <inertia ixx="${(1/12) * mass * (y*y+z*z)}" ixy="0.0" ixz="0.0"
-                    iyy="${(1/12) * mass * (x*x+z*z)}" iyz="0.0"
-                    izz="${(1/12) * mass * (x*x+y*y)}" />
+                     iyy="${(1/12) * mass * (x*x+z*z)}" iyz="0.0"
+                     izz="${(1/12) * mass * (x*x+y*y)}"/>
         </inertial>
     </xacro:macro>
@@ -24,8 +24,8 @@
         <inertial>
             <xacro:insert_block name="origin"/>
-            <mass value="${mass}" />
+            <mass value="${mass}"/>
             <inertia ixx="${(1/12) * mass * (3*radius*radius + length*length)}" ixy="0.0" ixz="0.0"
-                    iyy="${(1/12) * mass * (3*radius*radius + length*length)}" iyz="0.0"
-                    izz="${(1/2) * mass * (radius*radius)}" />
+                     iyy="${(1/12) * mass * (3*radius*radius + length*length)}" iyz="0.0"
+                     izz="${(1/2) * mass * (radius*radius)}"/>
         </inertial>
     </xacro:macro>

File: sec_test_dev_ws/src/sec_description/description/robot_core.xacro (robot description, xacro)
@@ -2,18 +2,4 @@
 <robot xmlns:xacro="http://ros.org/wiki/xacro">
     <xacro:include filename="inertial_macros.xacro"/>
-    <!-- Define robot constants -->
-    <!-- Unit -->
-    <xacro:property name="chassis_length" value="0.5"/> <!--X-->
-    <xacro:property name="chassis_width" value="0.5"/> <!--Y-->
-    <xacro:property name="chassis_height" value="0.5"/> <!--Z-->
-    <xacro:property name="chassis_mass" value="10"/>
-    <xacro:property name="wheel_radius" value="0.1"/>
-    <xacro:property name="wheel_length" value="0.1"/>
-    <xacro:property name="wheel_height_offset" value="0.03"/>
-    <xacro:property name="wheel_mass" value="10"/>
-    <!-- The difference between bottom middle of chassis and wheel position(s)-->
-    <xacro:property name="wheel_x_displacement" value="${chassis_length/4}"/>
-    <xacro:property name="wheel_y_displacement" value="${chassis_width/2+wheel_radius/2}"/>
-    <xacro:property name="wheel_z_displacement" value="0.03"/>
     <!-- Base Footprint -->
     <link name="base_link">
@@ -47,5 +33,5 @@
     <!-- Wheels -->
     <xacro:macro name="wheel" params="prefix l_r f_b">
-        <link name="${prefix}_wheel__link">
+        <link name="${prefix}_wheel_link">
             <visual>
                 <origin xyz="0 0 0" rpy="${pi/2} 0 0"/>
@@ -69,9 +55,9 @@
         <joint name="${prefix}_wheel_joint" type="continuous">
             <parent link="chassis"/>
-            <child link="${prefix}_link"/>
+            <child link="${prefix}_wheel_link"/>
             <origin xyz="${l_r*wheel_x_displacement} ${f_b*wheel_y_displacement} ${wheel_z_displacement}" rpy="0 0 0"/>
             <axis xyz="0 1 0"/>
         </joint>
-        <gazebo reference="${prefix}_wheel">
+        <gazebo reference="${prefix}_wheel_link">
             <material>Gazebo/Blue</material>
         </gazebo>

File: sec_test_dev_ws/src/sec_description/description/sec_description.urdf.xacro (robot description, xacro)
@@ -1,5 +1,19 @@
 <?xml version="1.0"?>
 <robot name="sec_bot" xmlns:xacro="http://ros.org/wiki/xacro">
+    <!-- Define robot constants -->
+    <!-- Unit -->
+    <xacro:property name="chassis_length" value="0.5"/> <!--X-->
+    <xacro:property name="chassis_width" value="0.5"/> <!--Y-->
+    <xacro:property name="chassis_height" value="0.5"/> <!--Z-->
+    <xacro:property name="chassis_mass" value="10"/>
+    <xacro:property name="wheel_radius" value="0.1"/>
+    <xacro:property name="wheel_length" value="0.1"/>
+    <xacro:property name="wheel_height_offset" value="0.03"/>
+    <xacro:property name="wheel_mass" value="10"/>
+    <!-- The difference between bottom middle of chassis and wheel position(s)-->
+    <xacro:property name="wheel_x_displacement" value="${chassis_length/4}"/>
+    <xacro:property name="wheel_y_displacement" value="${chassis_width/2+wheel_radius/2}"/>
+    <xacro:property name="wheel_z_displacement" value="0.03"/>
     <xacro:include filename="robot_core.xacro"/>
-    <>
+    <xacro:include filename="gazebo_control.xacro"/>
 </robot>
