Commit message: Test commit of simulation-based workspace that works in current environment

File: sec_test_dev_humble_ws/install/sec_description/share/sec_description/description/gazebo_control.xacro (robot description, xacro)
@@ -1 +1,27 @@
-/home/adenm/IEEE_SEC_HW_Competition/sec_test_dev_humble_ws/src/sec_description/description/gazebo_control.xacro
+<?xml version="1.0"?>
+<robot xmlns:xacro="http://www.ros.org/wiki/xacro">
+    <gazebo>
+        <plugin name="four_wheeled_robot_diff_drive" filename="libgazebo_ros_diff_drive.so">
+            <!-- Number of wheel pairs -->
+            <num_wheel_pairs>2</num_wheel_pairs>
+            <!-- wheels0 -->
+            <left_joint>f_l_wheel_joint</left_joint>
+            <right_joint>f_r_wheel_joint</right_joint>
+            <!-- wheels1-->
+            <left_joint>b_l_wheel_joint</left_joint>
+            <right_joint>b_r_wheel_joint</right_joint>
+            <!-- kinematics -->
+            <wheel_separation>${chassis_width}</wheel_separation>
+            <wheel_diameter>${wheel_radius*2}</wheel_diameter>
+            <!-- limits -->
+            <max_wheel_torque>200</max_wheel_torque>
+            <max_wheel_acceleration>10.0</max_wheel_acceleration>
+            <!-- output -->
+            <publish_odom>true</publish_odom>
+            <publish_odom_tf>true</publish_odom_tf>
+            <publish_wheel_tf>true</publish_wheel_tf>
+            <odometry_frame>odom</odometry_frame>
+            <robot_base_frame>base_link</robot_base_frame>
+        </plugin>
+    </gazebo>
+</robot>

File: sec_test_dev_humble_ws/install/sec_description/share/sec_description/description/gazebo_control_test.xacro (robot description, xacro)
@@ -1 +1,45 @@
-/home/adenm/IEEE_SEC_HW_Competition/sec_test_dev_humble_ws/src/sec_description/description/gazebo_control_test.xacro
+<?xml version="1.0"?>
+<robot xmlns:xacro="http://www.ros.org/wiki/xacro">
+    <gazebo>
+        <plugin name="skid_steer_drive_controller" filename="libgazebo_ros_skid_steer_drive.so">
+            <updateRate>100.0</updateRate>
+            <robotNamespace>/</robotNamespace>
+            <leftFrontJoint>f_l_wheel_joint</leftFrontJoint>
+            <rightFrontJoint>f_r_wheel_joint</rightFrontJoint>
+            <leftRearJoint>b_l_wheel_joint</leftRearJoint>
+            <rightRearJoint>b_r_wheel_joint</rightRearJoint>
+            <wheelSeparation>${chassis_length}</wheelSeparation>
+            <wheelDiameter>${wheel_radius*2}</wheelDiameter>
+            <robotBaseFrame>base_link</robotBaseFrame>
+            <torque>20</torque>
+            <topicName>cmd_vel</topicName>
+            <broadcastTF>true</broadcastTF>
+        </plugin>
+    </gazebo>
+    <gazebo>
+        <plugin name="four_wheeled_robot_diff_drive" filename="libgazebo_ros_skid_steer_drive.so">
+            <!-- Number of wheel pairs -->
+            <num_wheel_pairs>2</num_wheel_pairs>
+            <!-- wheels0 -->
+            <left_joint>f_l_wheel_joint</left_joint>
+            <right_joint>f_r_wheel_joint</right_joint>
+            <!-- wheels1-->
+            <left_joint>b_l_wheel_joint</left_joint>
+            <right_joint>b_r_wheel_joint</right_joint>
+            <!-- kinematics -->
+            <wheel_separation>"${chassis_width}"</wheel_separation>
+            <wheel_separation>"${chassis_width}"</wheel_separation>
+            <wheel_diameter>${wheel_radius*2}</wheel_diameter>
+            <wheel_diameter>${wheel_radius*2}</wheel_diameter>
+            <!-- limits -->
+            <max_wheel_torque>200</max_wheel_torque>
+            <max_wheel_acceleration>10.0</max_wheel_acceleration>
+            <!-- output -->
+            <publish_odom>true</publish_odom>
+            <publish_odom_tf>true</publish_odom_tf>
+            <publish_wheel_tf>true</publish_wheel_tf>
+            <odometry_frame>odom</odometry_frame>
+            <robot_base_frame>base_link</robot_base_frame>
+        </plugin>
+    </gazebo>
+</robot>

File: sec_test_dev_humble_ws/install/sec_description/share/sec_description/description/inertial_macros.xacro (robot description, xacro)
@@ -1 +1,32 @@
-/home/adenm/IEEE_SEC_HW_Competition/sec_test_dev_humble_ws/src/sec_description/description/inertial_macros.xacro
+<?xml version="1.0"?>
+<robot xmlns:xacro="http://www.ros.org/wiki/xacro">
+    <!-- Specify some standard inertial calculations https://en.wikipedia.org/wiki/List_of_moments_of_inertia -->
+    <!-- These make use of xacro's mathematical functionality -->
+    <xacro:macro name="inertial_sphere" params="mass radius *origin">
+        <inertial>
+            <xacro:insert_block name="origin"/>
+            <mass value="${mass}"/>
+            <inertia ixx="${(2/5) * mass * (radius*radius)}" ixy="0.0" ixz="0.0"
+                     iyy="${(2/5) * mass * (radius*radius)}" iyz="0.0"
+                     izz="${(2/5) * mass * (radius*radius)}"/>
+        </inertial>
+    </xacro:macro>
+    <xacro:macro name="inertial_box" params="mass x y z *origin">
+        <inertial>
+            <xacro:insert_block name="origin"/>
+            <mass value="${mass}"/>
+            <inertia ixx="${(1/12) * mass * (y*y+z*z)}" ixy="0.0" ixz="0.0"
+                     iyy="${(1/12) * mass * (x*x+z*z)}" iyz="0.0"
+                     izz="${(1/12) * mass * (x*x+y*y)}"/>
+        </inertial>
+    </xacro:macro>
+    <xacro:macro name="inertial_cylinder" params="mass length radius *origin">
+        <inertial>
+            <xacro:insert_block name="origin"/>
+            <mass value="${mass}"/>
+            <inertia ixx="${(1/12) * mass * (3*radius*radius + length*length)}" ixy="0.0" ixz="0.0"
+                     iyy="${(1/12) * mass * (3*radius*radius + length*length)}" iyz="0.0"
+                     izz="${(1/2) * mass * (radius*radius)}"/>
+        </inertial>
+    </xacro:macro>
+</robot>

File: sec_test_dev_humble_ws/install/sec_description/share/sec_description/description/robot_core.xacro (robot description, xacro)
@@ -1 +1,69 @@
-/home/adenm/IEEE_SEC_HW_Competition/sec_test_dev_humble_ws/src/sec_description/description/robot_core.xacro
+<?xml version="1.0"?>
+<robot xmlns:xacro="http://ros.org/wiki/xacro">
+    <xacro:include filename="inertial_macros.xacro"/>
+    <!-- Base Footprint -->
+    <link name="base_link">
+    </link>
+    <!-- Robot Base -->
+    <link name="chassis">
+        <visual>
+            <origin xyz="0 0 ${chassis_height/2}" rpy="0 0 0"/>
+            <geometry>
+                <box size="${chassis_length} ${chassis_width} ${chassis_height}"/>
+            </geometry>
+            <material name="Cyan">
+                <color rgba="0 1.0 1.0 1.0"/>
+            </material>
+        </visual>
+        <collision>
+            <origin xyz="0 0 ${chassis_height/2}" rpy="0 0 0"/>
+            <geometry>
+                <box size="${chassis_length} ${chassis_width} ${chassis_height}"/>
+            </geometry>
+        </collision>
+        <xacro:inertial_box mass="${chassis_mass}" x="${chassis_length}" y="${chassis_width}" z="${chassis_height}">
+            <origin xyz="0 0 ${chassis_height/2}" rpy="0 0 0"/>
+        </xacro:inertial_box>
+    </link>
+    <joint name="base_joint" type="fixed">
+        <parent link="base_link"/>
+        <child link="chassis"/>
+        <origin xyz="0.0 0.0 ${wheel_radius/2}" rpy="0 0 0"/>
+    </joint>
+    <!-- Wheels -->
+    <xacro:macro name="wheel" params="prefix l_r f_b">
+        <link name="${prefix}_wheel_link">
+            <visual>
+                <origin xyz="0 0 0" rpy="${pi/2} 0 0"/>
+                <geometry>
+                    <cylinder radius="${wheel_radius}" length="${wheel_length}"/>
+                </geometry>
+                <material name="Gray">
+                    <color rgba="0.5 0.5 0.5 1.0"/>
+                </material>
+            </visual>
+            <collision>
+                <origin xyz="0 0 0" rpy="${pi/2} 0 0"/>
+                <geometry>
+                    <cylinder radius="${wheel_radius}" length="${wheel_length}"/>
+                </geometry>
+            </collision>
+            <xacro:inertial_cylinder mass="${wheel_mass}" length="${wheel_length}" radius="${wheel_radius}">
+                <origin xyz="0 0 0" rpy="${pi/2} 0 0"/>
+            </xacro:inertial_cylinder>
+        </link>
+        <joint name="${prefix}_wheel_joint" type="continuous">
+            <parent link="chassis"/>
+            <child link="${prefix}_wheel_link"/>
+            <origin xyz="${l_r*wheel_x_displacement} ${f_b*wheel_y_displacement} ${wheel_z_displacement}" rpy="0 0 0"/>
+            <axis xyz="0 1 0"/>
+        </joint>
+        <gazebo reference="${prefix}_wheel_link">
+            <material>Gazebo/Blue</material>
+        </gazebo>
+    </xacro:macro>
+    <xacro:wheel prefix="b_l" l_r="-1" f_b="1" />
+    <xacro:wheel prefix="b_r" l_r="-1" f_b="-1" />
+    <xacro:wheel prefix="f_l" l_r="1"  f_b="1" />
+    <xacro:wheel prefix="f_r" l_r="1"  f_b="-1" />
+</robot>

File: sec_test_dev_humble_ws/install/sec_description/share/sec_description/description/sec_description.urdf.xacro (robot description, xacro)
@@ -1 +1,19 @@
-/home/adenm/IEEE_SEC_HW_Competition/sec_test_dev_humble_ws/src/sec_description/description/sec_description.urdf.xacro
+<?xml version="1.0"?>
+<robot name="sec_bot" xmlns:xacro="http://ros.org/wiki/xacro">
+    <!-- Define robot constants -->
+    <!-- Unit -->
+    <xacro:property name="chassis_length" value="0.5"/> <!--X-->
+    <xacro:property name="chassis_width" value="0.5"/> <!--Y-->
+    <xacro:property name="chassis_height" value="0.5"/> <!--Z-->
+    <xacro:property name="chassis_mass" value="10"/>
+    <xacro:property name="wheel_radius" value="0.1"/>
+    <xacro:property name="wheel_length" value="0.1"/>
+    <xacro:property name="wheel_height_offset" value="0.03"/>
+    <xacro:property name="wheel_mass" value="10"/>
+    <!-- The difference between bottom middle of chassis and wheel position(s)-->
+    <xacro:property name="wheel_x_displacement" value="${chassis_length/4}"/>
+    <xacro:property name="wheel_y_displacement" value="${chassis_width/2+wheel_radius/2}"/>
+    <xacro:property name="wheel_z_displacement" value="0.03"/>
+    <xacro:include filename="robot_core.xacro"/>
+    <xacro:include filename="gazebo_control.xacro"/>
+</robot>

File: sec_test_dev_humble_ws/install/sec_description/share/sec_description/description/sec_description_final.urdf.xacro (robot description, xacro)
@@ -1,5 +1,5 @@
 <?xml version="1.0" ?>
 <!-- =================================================================================== -->
-<!-- |    This document was autogenerated by xacro from /home/adenm/IEEE_SEC_HW_Competition/sec_test_dev_humble_ws/install/sec_description/share/sec_description/description/sec_description.urdf.xacro | -->
+<!-- |    This document was autogenerated by xacro from /home/orion/IEEE_SEC_HW_Competition/sec_test_dev_humble_ws/install/sec_description/share/sec_description/description/sec_description.urdf.xacro | -->
 <!-- |    EDITING THIS FILE BY HAND IS NOT RECOMMENDED                                 | -->
 <!-- =================================================================================== -->
@@ -173,5 +173,5 @@
 			<right_joint>b_r_wheel_joint</right_joint>
 			<!-- kinematics -->
-			<wheel_separation>&quot;0.5&quot;</wheel_separation>
+			<wheel_separation>0.5</wheel_separation>
 			<wheel_diameter>0.2</wheel_diameter>
 			<!-- limits -->
@@ -183,5 +183,5 @@
 			<publish_wheel_tf>true</publish_wheel_tf>
 			<odometry_frame>odom</odometry_frame>
-			<robot_base_frame>chassis</robot_base_frame>
+			<robot_base_frame>base_link</robot_base_frame>
 		</plugin>
 	</gazebo>

File: sec_test_dev_humble_ws/src/sec_description/description/gazebo_control.xacro (robot description, xacro)
@@ -12,5 +12,5 @@
             <right_joint>b_r_wheel_joint</right_joint>
             <!-- kinematics -->
-            <wheel_separation>"${chassis_width}"</wheel_separation>
+            <wheel_separation>${chassis_width}</wheel_separation>
             <wheel_diameter>${wheel_radius*2}</wheel_diameter>
             <!-- limits -->
@@ -22,5 +22,5 @@
             <publish_wheel_tf>true</publish_wheel_tf>
             <odometry_frame>odom</odometry_frame>
-            <robot_base_frame>chassis</robot_base_frame>
+            <robot_base_frame>base_link</robot_base_frame>
         </plugin>
     </gazebo>
