Commit message: added camera sensor simulation on gazebo

File: sec_test_dev_humble_ws/install/sec_description/share/sec_description/description/sec_description.urdf.xacro (robot description, xacro)
@@ -15,5 +15,11 @@
     <xacro:property name="wheel_y_displacement" value="${chassis_width/2+wheel_radius/2}"/>
     <xacro:property name="wheel_z_displacement" value="0.03"/>
+    <xacro:property name="camera_x" value="0.010"/>
+    <xacro:property name="camera_y" value="0.03"/>
+    <xacro:property name="camera_z" value="0.03"/>
+    <xacro:property name="camera_y" value="0.03"/>
+    <xacro:property name="camera_fov" value="1.089"/>
     <xacro:include filename="robot_core.xacro"/>
     <xacro:include filename="gazebo_control.xacro"/>
+    <xacro:include filename="camera.xacro"/>
 </robot>

File: sec_test_dev_humble_ws/install/sec_description/share/sec_description/description/sec_description_final.urdf.xacro (robot description, xacro)
@@ -186,3 +186,47 @@
 		</plugin>
 	</gazebo>
+	<joint name="camera_joint" type="fixed">
+		<parent link="chassis"/>
+		<child link="camera_link"/>
+		<origin rpy="0 0 0" xyz="0.255 0 0.25"/>
+	</joint>
+	<link name="camera_link">
+		<visual>
+			<geometry>
+				<box size="0.01 0.03 0.03"/>
+			</geometry>
+			<material name="Gray">
+				<color rgba="0.5 0.5 0.5 1.0"/>
+			</material>
+		</visual>
+	</link>
+	<joint name="camera_optical_joint" type="fixed">
+		<parent link="camera_link"/>
+		<child link="camera_link_optical"/>
+		<origin rpy="-1.5707963267948966 0 -1.5707963267948966" xyz="0 0 0"/>
+	</joint>
+	<link name="camera_link_optical"/>
+	<gazebo reference="camera_link">
+		<material>Gazebo/Red</material>
+		<sensor name="camera" type="camera">
+			<pose> 0 0 0 0 0 0 </pose>
+			<visualize>true</visualize>
+			<update_rate>10</update_rate>
+			<camera>
+				<horizontal_fov>1.089</horizontal_fov>
+				<image>
+					<format>R8G8B8</format>
+					<width>640</width>
+					<height>480</height>
+				</image>
+				<clip>
+					<near>0.05</near>
+					<far>8.0</far>
+				</clip>
+			</camera>
+			<plugin filename="libgazebo_ros_camera.so" name="camera_controller">
+				<frame_name>camera_link_optical</frame_name>
+			</plugin>
+		</sensor>
+	</gazebo>
 </robot>

Commit message: Added imu simulation to gazebo. Use ros2 topic echo /imu/data to see published data

File: sec_test_dev_humble_ws/install/sec_description/share/sec_description/description/sec_description.urdf.xacro (robot description, xacro)
@@ -20,6 +20,10 @@
     <xacro:property name="camera_y" value="0.03"/>
     <xacro:property name="camera_fov" value="1.089"/>
+    <xacro:property name="imu_length" value="0.05"/>
+    <xacro:property name="imu_width" value="0.05"/>
+    <xacro:property name="imu_height" value="0.02"/>
     <xacro:include filename="robot_core.xacro"/>
     <xacro:include filename="gazebo_control.xacro"/>
     <xacro:include filename="camera.xacro"/>
+    <xacro:include filename="imu.xacro"/>
 </robot>

File: sec_test_dev_humble_ws/install/sec_description/share/sec_description/description/sec_description_final.urdf.xacro (robot description, xacro)
@@ -230,3 +230,86 @@
 		</sensor>
 	</gazebo>
+	<joint name="imu_joint" type="fixed">
+		<parent link="chassis"/>
+		<child link="imu_link"/>
+		<origin rpy="0 0 0" xyz="0 0 0.51"/>
+	</joint>
+	<link name="imu_link">
+		<visual>
+			<geometry>
+				<box size="0.05 0.05 0.02"/>
+			</geometry>
+			<material name="Gray">
+				<color rgba="0.5 0.5 0.5 1.0"/>
+			</material>
+		</visual>
+	</link>
+	<!--        <gazebo reference="imu_link">
+            <material>Gazebo/Red</material>
+            <sensor name="imu_sensor" type="imu">
+                <pose>0 0 0 0 0 0</pose>
+                <visualize>true</visualize>
+                <update_rate>10</update_rate>
+                <always_on>true</always_on>
+                <topic>imu</topic>
+                <plugin name="imu_plugin" filename="libgazebo_ros_imu_sensor.so">
+                    <frame_name>imu_link</frame_name>
+                </plugin>
+            </sensor>
+        </gazebo>-->
+	<gazebo reference="imu_link">
+		<sensor name="br_imu" type="imu">
+			<always_on>true</always_on>
+			<update_rate>100</update_rate>
+			<imu>
+				<angular_velocity>
+					<x>
+						<noise type="gaussian">
+							<mean>0.0</mean>
+							<stddev>2e-4</stddev>
+						</noise>
+					</x>
+					<y>
+						<noise type="gaussian">
+							<mean>0.0</mean>
+							<stddev>2e-4</stddev>
+						</noise>
+					</y>
+					<z>
+						<noise type="gaussian">
+							<mean>0.0</mean>
+							<stddev>2e-4</stddev>
+						</noise>
+					</z>
+				</angular_velocity>
+				<linear_acceleration>
+					<x>
+						<noise type="gaussian">
+							<mean>0.0</mean>
+							<stddev>1.7e-2</stddev>
+						</noise>
+					</x>
+					<y>
+						<noise type="gaussian">
+							<mean>0.0</mean>
+							<stddev>1.7e-2</stddev>
+						</noise>
+					</y>
+					<z>
+						<noise type="gaussian">
+							<mean>0.0</mean>
+							<stddev>1.7e-2</stddev>
+						</noise>
+					</z>
+				</linear_acceleration>
+			</imu>
+			<plugin filename="libgazebo_ros_imu_sensor.so" name="bytes_imu">
+				<ros>
+					<namespace>imu</namespace>
+					<remapping>~/out:=data</remapping>
+				</ros>
+				<initial_orientation_as_reference>false</initial_orientation_as_reference>
+			</plugin>
+		</sensor>
+	</gazebo>
 </robot>
