Commit message: removed old and personal code

File: sec_test_dev_humble_ws/install/sec_description/share/sec_description/description/sec_description_final.urdf.xacro (robot description, xacro)
@@ -245,17 +245,4 @@
 		</visual>
 	</link>
-	<!--        <gazebo reference="imu_link">
-            <material>Gazebo/Red</material>
-            <sensor name="imu_sensor" type="imu">
-                <pose>0 0 0 0 0 0</pose>
-                <visualize>true</visualize>
-                <update_rate>10</update_rate>
-                <always_on>true</always_on>
-                <topic>imu</topic>
-                <plugin name="imu_plugin" filename="libgazebo_ros_imu_sensor.so">
-                    <frame_name>imu_link</frame_name>
-                </plugin>
-            </sensor>
-        </gazebo>-->
 	<gazebo reference="imu_link">
 		<sensor name="br_imu" type="imu">
@@ -309,5 +296,5 @@
 					<remapping>~/out:=data</remapping>
 				</ros>
-				<initial_orientation_as_reference>false</initial_orientation_as_reference>
+				<initial_orientation_as_reference>true</initial_orientation_as_reference>
 			</plugin>
 		</sensor>
