Commit message: added lidar to simulation

File: sec_test_dev_humble_ws/install/sec_description/share/sec_description/description/camera.xacro (robot description, xacro)
@@ -15,4 +15,7 @@
                 </material>
             </visual>
+        <xacro:inertial_box mass=".7" x="${camera_x}" y="${camera_y}" z="${camera_z}">
+            <origin xyz="0 0 0" rpy="0 0 0"/>
+        </xacro:inertial_box>
         </link>
         <joint name="camera_optical_joint" type="fixed">

File: sec_test_dev_humble_ws/install/sec_description/share/sec_description/description/imu.xacro (robot description, xacro)
@@ -4,16 +4,19 @@
             <parent link="chassis"/>
             <child link="imu_link"/>
-            <origin xyz="0 0 ${chassis_height+(imu_height/2)}" rpy="0 0 0"/>
+            <origin xyz="-0.2 0 ${chassis_height+(imu_height/2)}" rpy="0 0 0"/>
         </joint>
-        <link name="imu_link">
-            <visual>
-                <geometry>
-                    <box size="${imu_length} ${imu_width} ${imu_height}"/>
-                </geometry>
-                <material name="Gray">
-                    <color rgba="0.5 0.5 0.5 1.0"/>
-                </material>
-            </visual>
-        </link>
+    <link name="imu_link">
+        <visual>
+            <geometry>
+                <box size="${imu_length} ${imu_width} ${imu_height}"/>
+            </geometry>
+            <material name="Gray">
+                <color rgba="0.5 0.5 0.5 1.0"/>
+            </material>
+        </visual>
+        <xacro:inertial_box mass=".15" x="${imu_width}" y="${imu_length}" z="${imu_height}">
+            <origin xyz="0 0 0" rpy="0 0 0"/>
+        </xacro:inertial_box>
+    </link>
     <gazebo reference="imu_link">
         <sensor name="br_imu" type="imu">

File: sec_test_dev_humble_ws/install/sec_description/share/sec_description/description/sec_description.urdf.xacro (robot description, xacro)
@@ -18,12 +18,14 @@
     <xacro:property name="camera_y" value="0.03"/>
     <xacro:property name="camera_z" value="0.03"/>
-    <xacro:property name="camera_y" value="0.03"/>
     <xacro:property name="camera_fov" value="1.089"/>
     <xacro:property name="imu_length" value="0.05"/>
     <xacro:property name="imu_width" value="0.05"/>
     <xacro:property name="imu_height" value="0.02"/>
+    <xacro:property name="lidar_radius" value="0.05"/>
+    <xacro:property name="lidar_length" value="0.04"/>
     <xacro:include filename="robot_core.xacro"/>
     <xacro:include filename="gazebo_control.xacro"/>
     <xacro:include filename="camera.xacro"/>
     <xacro:include filename="imu.xacro"/>
+    <xacro:include filename="lidar.xacro"/>
 </robot>

File: sec_test_dev_humble_ws/install/sec_description/share/sec_description/description/sec_description_final.urdf.xacro (robot description, xacro)
@@ -200,4 +200,9 @@
 			</material>
 		</visual>
+		<inertial>
+			<origin rpy="0 0 0" xyz="0 0 0"/>
+			<mass value="0.7"/>
+			<inertia ixx="0.00010499999999999999" ixy="0.0" ixz="0.0" iyy="5.8333333333333326e-05" iyz="0.0" izz="5.8333333333333326e-05"/>
+		</inertial>
 	</link>
 	<joint name="camera_optical_joint" type="fixed">
@@ -233,5 +238,5 @@
 		<parent link="chassis"/>
 		<child link="imu_link"/>
-		<origin rpy="0 0 0" xyz="0 0 0.51"/>
+		<origin rpy="0 0 0" xyz="-0.2 0 0.51"/>
 	</joint>
 	<link name="imu_link">
@@ -244,4 +249,9 @@
 			</material>
 		</visual>
+		<inertial>
+			<origin rpy="0 0 0" xyz="0 0 0"/>
+			<mass value="0.15"/>
+			<inertia ixx="3.625000000000001e-05" ixy="0.0" ixz="0.0" iyy="3.625000000000001e-05" iyz="0.0" izz="6.25e-05"/>
+		</inertial>
 	</link>
 	<gazebo reference="imu_link">
@@ -300,3 +310,52 @@
 		</sensor>
 	</gazebo>
+	<joint name="lidar_joint" type="fixed">
+		<parent link="chassis"/>
+		<child link="lidar_link"/>
+		<origin rpy="0 0 0" xyz="0 0 0.51"/>
+	</joint>
+	<link name="lidar_link">
+		<visual>
+			<geometry>
+				<cylinder length="0.04" radius="0.05"/>
+			</geometry>
+			<material name="Gray">
+				<color rgba="0.5 0.5 0.5 1.0"/>
+			</material>
+		</visual>
+		<inertial>
+			<origin rpy="0 0 0" xyz="0 0 0"/>
+			<mass value="0.1"/>
+			<inertia ixx="7.583333333333335e-05" ixy="0.0" ixz="0.0" iyy="7.583333333333335e-05" iyz="0.0" izz="0.00012500000000000003"/>
+		</inertial>
+	</link>
+	<gazebo reference="lidar_link">
+		<sensor name="laser" type="ray">
+			<visualize>true</visualize>
+			<pose>0.0 0 0.0 0 0 0</pose>
+			<update_rate>10</update_rate>
+			<ray>
+				<scan>
+					<horizontal>
+						<samples>360</samples>
+						<resolution>1</resolution>
+						<min_angle>-3.14</min_angle>
+						<max_angle>3.14</max_angle>
+					</horizontal>
+				</scan>
+				<range>
+					<min>0.3</min>
+					<max>12</max>
+					<resolution>0.01</resolution>
+				</range>
+			</ray>
+			<plugin filename="libgazebo_ros_ray_sensor.so" name="laser_controller">
+				<ros>
+					<argument>~/out:=scan</argument>
+				</ros>
+				<output_type>sensor_msgs/LaserScan</output_type>
+				<frame_name>lidar_link</frame_name>
+			</plugin>
+		</sensor>
+	</gazebo>
 </robot>
