Commit message: partial ros2_control gazebo implementation, needs to be debugged with launch file

File: sec_test_dev_humble_ws/src/sec_description/description/sec_description.urdf.xacro (robot description, xacro)
@@ -7,5 +7,5 @@
     <xacro:property name="chassis_height" value="0.5"/> <!--Z-->
     <xacro:property name="chassis_mass" value="10"/>
-    <xacro:property name="wheel_radius" value="0.1"/>
+    <xacro:property name="wheel_radius" value="0.1"/> <!-- Update wheel radius paramter in controllers.yaml as well-->
     <xacro:property name="wheel_length" value="0.1"/>
     <xacro:property name="wheel_height_offset" value="0.03"/>
@@ -13,7 +13,8 @@
     <!-- The difference between bottom middle of chassis and wheel position(s)-->
     <xacro:property name="wheel_x_displacement" value="${chassis_length/4}"/>
-    <xacro:property name="wheel_y_displacement" value="${chassis_width/2+wheel_radius/2}"/>
+    <xacro:property name="wheel_y_displacement" value="${chassis_width/2+wheel_radius/2}"/> <!-- Update wheel separation paramter in controllers.yaml as well-->
     <xacro:property name="wheel_z_displacement" value="0.03"/>
     <xacro:include filename="robot_core.xacro"/>
-    <xacro:include filename="gazebo_control.xacro"/>
+    <!-- xacro:include filename="gazebo_control.xacro"/ -->
+    <xacro:include filename="ros2_control.xacro"/>
 </robot>
