Commit message: changed wheel collision to sphere to reduce drift, more to do

File: sec_test_dev_humble_ws/src/sec_description/description/robot_core.xacro (robot description, xacro)
@@ -2,8 +2,21 @@
 <robot xmlns:xacro="http://ros.org/wiki/xacro">
     <xacro:include filename="inertial_macros.xacro"/>
-    <!-- Base Footprint -->
+    <!-- Base Link -->
     <link name="base_link">
     </link>
-    <!-- Robot Base -->
+    <!-- Base Footprint Link-->
+    <joint name="base_footprint_joint" type="fixed">
+        <parent link="base_link"/>
+        <child link="base_footprint"/>
+        <origin xyz="0 0 0" rpy="0 0 0"/>
+    </joint>
+    <link name="base_footprint">
+    </link>
+    <!-- Chassis -->
+    <joint name="chassis_joint" type="fixed">
+        <parent link="base_link"/>
+        <child link="chassis"/>
+        <origin xyz="0.0 0.0 ${wheel_radius/2}" rpy="0 0 0"/>
+    </joint>
     <link name="chassis">
         <visual>
@@ -26,11 +39,12 @@
         </xacro:inertial_box>
     </link>
-    <joint name="base_joint" type="fixed">
-        <parent link="base_link"/>
-        <child link="chassis"/>
-        <origin xyz="0.0 0.0 ${wheel_radius/2}" rpy="0 0 0"/>
-    </joint>
     <!-- Wheels -->
     <xacro:macro name="wheel" params="prefix l_r f_b">
+        <joint name="${prefix}_wheel_joint" type="continuous">
+            <parent link="chassis"/>
+            <child link="${prefix}_wheel_link"/>
+            <origin xyz="${l_r*wheel_x_displacement} ${f_b*wheel_y_displacement} ${wheel_z_displacement}" rpy="0 0 0"/>
+            <axis xyz="0 1 0"/>
+        </joint>
         <link name="${prefix}_wheel_link">
             <visual>
@@ -46,5 +60,5 @@
                 <origin xyz="0 0 0" rpy="${pi/2} 0 0"/>
                 <geometry>
-                    <cylinder radius="${wheel_radius}" length="${wheel_length}"/>
+                    <sphere radius="${wheel_radius}"/>
                 </geometry>
             </collision>
@@ -53,10 +67,4 @@
             </xacro:inertial_cylinder>
         </link>
-        <joint name="${prefix}_wheel_joint" type="continuous">
-            <parent link="chassis"/>
-            <child link="${prefix}_wheel_link"/>
-            <origin xyz="${l_r*wheel_x_displacement} ${f_b*wheel_y_displacement} ${wheel_z_displacement}" rpy="0 0 0"/>
-            <axis xyz="0 1 0"/>
-        </joint>
         <gazebo reference="${prefix}_wheel_link">
             <material>Gazebo/Blue</material>

File: sec_test_dev_humble_ws/src/sec_description/description/sec_description.urdf.xacro (robot description, xacro)
@@ -13,5 +13,5 @@
     <!-- The difference between bottom middle of chassis and wheel position(s)-->
     <xacro:property name="wheel_x_displacement" value="${chassis_length/4}"/>
-    <xacro:property name="wheel_y_displacement" value="${chassis_width/2+wheel_radius/2}"/> <!-- Update wheel separation paramter in controllers.yaml as well-->
+    <xacro:property name="wheel_y_displacement" value="${chassis_width/2+wheel_radius}"/> <!-- Update wheel separation paramter in controllers.yaml as well-->
     <xacro:property name="wheel_z_displacement" value="0.03"/>
     <xacro:include filename="robot_core.xacro"/>

Commit message: random inconsequential comment changes

File: sec_test_dev_humble_ws/src/sec_description/description/robot_core.xacro (robot description, xacro)
@@ -3,7 +3,6 @@
     <xacro:include filename="inertial_macros.xacro"/>
     <!-- Base Link -->
-    <link name="base_link">
-    </link>
-    <!-- Base Footprint Link-->
+    <link name="base_link"/>
+    <!--Base Footprint Link-->
     <joint name="base_footprint_joint" type="fixed">
         <parent link="base_link"/>

Commit message: fixed mesh scaling, initial pose, and robot scale issues

File: sec_test_dev_humble_ws/src/sec_description/description/robot_core.xacro (robot description, xacro)
@@ -16,5 +16,5 @@
         <parent link="base_link"/>
         <child link="chassis"/>
-        <origin xyz="0.0 0.0 ${wheel_radius/2}" rpy="0 0 0"/>
+        <origin xyz="0.0 0.0 ${wheel_radius/2 + chassis_z_offset}" rpy="0 0 0"/>
     </joint>
     <link name="chassis">

File: sec_test_dev_humble_ws/src/sec_description/description/sec_description.urdf.xacro (robot description, xacro)
@@ -4,12 +4,12 @@
     <xacro:arg name="sim_mode" default="true"/>
     <!-- Define robot constants -->
-    <!-- Unit -->
-    <xacro:property name="chassis_length" value="0.5"/> <!--X-->
-    <xacro:property name="chassis_width" value="0.5"/> <!--Y-->
-    <xacro:property name="chassis_height" value="0.5"/> <!--Z-->
-    <xacro:property name="chassis_mass" value="10"/>
-    <xacro:property name="wheel_radius" value="0.1"/> <!-- Update wheel radius paramter in controllers.yaml as well-->
-    <xacro:property name="wheel_length" value="0.1"/>
-    <xacro:property name="wheel_height_offset" value="0.03"/>
+    <!-- Meters -->
+    <xacro:property name="chassis_length" value="0.205"/> <!--X-->
+    <xacro:property name="chassis_width" value="0.205"/> <!--Y-->
+    <xacro:property name="chassis_height" value="0.205"/> <!--Z-->
+    <xacro:property name="chassis_mass" value="10"/> <!--WHat is the unit for this?-->
+    <xacro:property name="chassis_z_offset" value="0.1"/> <!--Currently unused, going to try to implement for total height translation-->
+    <xacro:property name="wheel_radius" value="0.05"/> <!-- Update wheel radius paramter in controllers.yaml as well-->
+    <xacro:property name="wheel_length" value="0.025"/>
     <xacro:property name="wheel_mass" value="10"/>
     <!-- The difference between bottom middle of chassis and wheel position(s)-->
