Commit message: fixed wheel width added slam dependencies

File: src_ws/src/secbot_description/description/robot_core_hw.xacro (robot description, xacro)
@@ -13,5 +13,5 @@
     <!-- The difference between bottom middle of chassis and wheel position(s)-->
     <xacro:property name="wheel_x_displacement" value="0.0"/>
-    <xacro:property name="wheel_y_displacement" value="${chassis_width/2+wheel_radius}"/> <!-- Update wheel separation paramter in controllers.yaml as well-->
+    <xacro:property name="wheel_y_displacement" value="0.115"/> <!-- Update wheel separation paramter in controllers.yaml as well-->
     <xacro:property name="wheel_z_displacement" value="0.03"/>
     <!-- Base Link -->
@@ -55,5 +55,5 @@
         <parent link="chassis"/>
         <child link="left_wheel"/>
-        <origin xyz="${-1*wheel_x_displacement} ${0} ${wheel_z_displacement}" rpy="0 0 0"/>
+        <origin xyz="${-1*wheel_x_displacement} ${-1*wheel_y_displacement} ${wheel_z_displacement}" rpy="0 0 0"/>
         <axis xyz="0 1 0"/>
     </joint>
@@ -81,5 +81,5 @@
         <parent link="chassis"/>
         <child link="right_wheel"/>
-        <origin xyz="${wheel_x_displacement} ${0} ${wheel_z_displacement}" rpy="0 0 0"/>
+        <origin xyz="${wheel_x_displacement} ${wheel_y_displacement} ${wheel_z_displacement}" rpy="0 0 0"/>
         <axis xyz="0 1 0"/>
     </joint>

Commit message: fixed urdf inconsistencies, launch errors, and smake build errors

File: src_ws/src/secbot_description/description/robot_core_hw.xacro (robot description, xacro)
@@ -52,11 +52,11 @@
     </link>
     <!-- Wheels -->
-    <joint name="$l_wheel_joints" type="continuous">
+    <joint name="l_wheel_joints" type="continuous">
         <parent link="chassis"/>
-        <child link="${prefix}_wheel_link"/>
-        <origin xyz="${l_r*wheel_x_displacement} ${f_b*wheel_y_displacement} ${wheel_z_displacement}" rpy="0 0 0"/>
+        <child link="l_wheel_link"/>
+        <origin xyz="${-1*wheel_x_displacement} ${0} ${wheel_z_displacement}" rpy="0 0 0"/>
         <axis xyz="0 1 0"/>
     </joint>
-    <link name="$l_wheel_link">
+    <link name="l_wheel_link">
         <visual>
             <origin xyz="0 0 0" rpy="${pi/2} 0 0"/>
@@ -78,11 +78,11 @@
         </xacro:inertial_cylinder>
     </link>
-    <joint name="$r_wheel_joints" type="continuous">
+    <joint name="r_wheel_joints" type="continuous">
         <parent link="chassis"/>
-        <child link="${prefix}_wheel_link"/>
-        <origin xyz="${l_r*wheel_x_displacement} ${f_b*wheel_y_displacement} ${wheel_z_displacement}" rpy="0 0 0"/>
+        <child link="r_wheel_link"/>
+        <origin xyz="${wheel_x_displacement} ${0} ${wheel_z_displacement}" rpy="0 0 0"/>
         <axis xyz="0 1 0"/>
     </joint>
-    <link name="$r_wheel_link">
+    <link name="r_wheel_link">
         <visual>
             <origin xyz="0 0 0" rpy="${pi/2} 0 0"/>

File: src_ws/src/secbot_description/description/ros2_control.xacro (robot description, xacro)
@@ -6,14 +6,14 @@
                 <plugin>diffdrive_arduino/DiffDriveArduinoHardware</plugin>
             </hardware>
-            <joint name="$l_wheel_joints" type="continuous">
+            <joint name="l_wheel_joints" type="continuous">
                 <parent link="chassis"/>
-                <child link="${prefix}_wheel_link"/>
-                <origin xyz="${l_r*wheel_x_displacement} ${f_b*wheel_y_displacement} ${wheel_z_displacement}" rpy="0 0 0"/>
+                <child link="l_wheel_link"/>
+                <origin xyz="${-1*wheel_x_displacement} ${0} ${wheel_z_displacement}" rpy="0 0 0"/>
                 <axis xyz="0 1 0"/>
             </joint>
-            <joint name="$r_wheel_joints" type="continuous">
+            <joint name="r_wheel_joints" type="continuous">
                 <parent link="chassis"/>
-                <child link="${prefix}_wheel_link"/>
-                <origin xyz="${l_r*wheel_x_displacement} ${f_b*wheel_y_displacement} ${wheel_z_displacement}" rpy="0 0 0"/>
+                <child link="r_wheel_link"/>
+                <origin xyz="${wheel_x_displacement} ${0} ${wheel_z_displacement}" rpy="0 0 0"/>
                 <axis xyz="0 1 0"/>
             </joint>

File: src_ws/src/secbot_description/description/sec_description.urdf.xacro (robot description, xacro)
@@ -12,7 +12,4 @@
     <xacro:property name="lidar_radius" value="0.05"/>
     <xacro:property name="lidar_length" value="0.04"/>
-    <xacro:include filename="camera.xacro"/>
-    <xacro:include filename="imu.xacro"/>
-    <xacro:include filename="lidar.xacro"/>
     <xacro:if value="$(arg sim_mode)">
         <xacro:include filename="robot_core_sim.xacro"/>
@@ -21,4 +18,7 @@
         <xacro:include filename="robot_core_hw.xacro" />
     </xacro:unless>
+    <xacro:include filename="camera.xacro"/>
+    <xacro:include filename="imu.xacro"/>
+    <xacro:include filename="lidar.xacro"/>
     <xacro:if value="$(arg use_ros2_control)">
         <xacro:include filename="ros2_control.xacro" />

Commit message: fixed nonav and hardware launch files

File: src_ws/src/secbot_description/description/robot_core_hw.xacro (robot description, xacro)
@@ -52,11 +52,11 @@
     </link>
     <!-- Wheels -->
-    <joint name="l_wheel_joints" type="continuous">
+    <joint name="b_l_wheel_joints" type="continuous">
         <parent link="chassis"/>
-        <child link="l_wheel_link"/>
+        <child link="b_l_wheel_link"/>
         <origin xyz="${-1*wheel_x_displacement} ${0} ${wheel_z_displacement}" rpy="0 0 0"/>
         <axis xyz="0 1 0"/>
     </joint>
-    <link name="l_wheel_link">
+    <link name="b_l_wheel_link">
         <visual>
             <origin xyz="0 0 0" rpy="${pi/2} 0 0"/>
@@ -78,11 +78,11 @@
         </xacro:inertial_cylinder>
     </link>
-    <joint name="r_wheel_joints" type="continuous">
+    <joint name="b_r_wheel_joints" type="continuous">
         <parent link="chassis"/>
-        <child link="r_wheel_link"/>
+        <child link="b_r_wheel_link"/>
         <origin xyz="${wheel_x_displacement} ${0} ${wheel_z_displacement}" rpy="0 0 0"/>
         <axis xyz="0 1 0"/>
     </joint>
-    <link name="r_wheel_link">
+    <link name="b_r_wheel_link">
         <visual>
             <origin xyz="0 0 0" rpy="${pi/2} 0 0"/>

File: src_ws/src/secbot_description/description/ros2_control.xacro (robot description, xacro)
@@ -1,4 +1,5 @@
 <?xml version="1.0"?>
 <robot xmlns:xacro="http://ros.org/wiki/xacro">
+<!--
     <xacro:unless value="$(arg sim_mode)">
         <ros2_control name="RealRobot" type="system">
@@ -19,5 +20,5 @@
             </joint>
         </ros2_control>
-        <!-- IMU sensor-->
+         IMU sensor-->
         <!-- <ros2_control name='da_imu' type='sensor'>
             <hardware>
@@ -29,5 +30,5 @@
                 STATE INTERFACES HERE
             </sensor>
-        </ros2_control>  -->
+        </ros2_control>
     </xacro:unless>
     <xacro:if value="$(arg sim_mode)">
@@ -70,8 +71,60 @@
         </ros2_control>
     </xacro:if>
+-->
+<ros2_control name='RealRobot' type='system'>
+            <hardware>
+                <plugin>diffdrive_arduino/DiffDriveArduinoHardware</plugin>
+                <param name="left_wheel_name">b_l_wheel_joint</param>
+                <param name="right_wheel_name">b_r_wheel_joint</param>
+                <param name="loop_rate">30</param>
+                <param name="device">/dev/ttyUSB1</param>
+                <param name="baud_rate">115200</param>
+                <param name="timeout_ms">1000</param>
+                <param name="enc_counts_per_rev">3436</param>
+                <param name="pid_p">20</param>
+                <param name="pid_d">12</param>
+                <param name="pid_i">0</param>
+                <param name="pid_o">50</param>
+            </hardware>
+            <joint name="b_l_wheel_joint">
+                <command_interface name="velocity">
+                    <param name="min">-10</param>
+                    <param name="max">10</param>
+                </command_interface>
+                <state_interface name="position" />
+                <state_interface name="velocity" />
+            </joint>
+            <joint name="b_r_wheel_joint">
+                <command_interface name="velocity">
+                    <param name="min">-10</param>
+                    <param name="max">10</param>
+                </command_interface>
+                <state_interface name="position" />
+                <state_interface name="velocity" />
+            </joint>
+<!--
+            <joint name="f_l_wheel_joint">
+                <command_interface name="velocity">
+                    <param name="min">-10</param>
+                    <param name="max">10</param>
+                </command_interface>
+                <state_interface name="position" />
+                <state_interface name="velocity" />
+            </joint>
+            <joint name="f_r_wheel_joint">
+                <command_interface name="velocity">
+                    <param name="min">-10</param>
+                    <param name="max">10</param>
+                </command_interface>
+                <state_interface name="position" />
+                <state_interface name="velocity" />
+            </joint>
+-->
+        </ros2_control>
+<!--
     <gazebo>
         <plugin filename="libgazebo_ros2_control.so" name="gazebo_ros2_control">
             <parameters>$(find secbot_description)/config/controllers.yaml</parameters>
         </plugin>
-    </gazebo>
+    </gazebo>-->
 </robot>

Commit message: big commit, just read through it

File: src_ws/src/secbot_description/description/robot_core_hw.xacro (robot description, xacro)
@@ -52,11 +52,11 @@
     </link>
     <!-- Wheels -->
-    <joint name="b_l_wheel_joints" type="continuous">
+    <joint name="left_wheel_joint" type="continuous">
         <parent link="chassis"/>
-        <child link="b_l_wheel_link"/>
+        <child link="left_wheel"/>
         <origin xyz="${-1*wheel_x_displacement} ${0} ${wheel_z_displacement}" rpy="0 0 0"/>
         <axis xyz="0 1 0"/>
     </joint>
-    <link name="b_l_wheel_link">
+    <link name="left_wheel">
         <visual>
             <origin xyz="0 0 0" rpy="${pi/2} 0 0"/>
@@ -78,11 +78,11 @@
         </xacro:inertial_cylinder>
     </link>
-    <joint name="b_r_wheel_joints" type="continuous">
+    <joint name="right_wheel_joint" type="continuous">
         <parent link="chassis"/>
-        <child link="b_r_wheel_link"/>
+        <child link="right_wheel"/>
         <origin xyz="${wheel_x_displacement} ${0} ${wheel_z_displacement}" rpy="0 0 0"/>
         <axis xyz="0 1 0"/>
     </joint>
-    <link name="b_r_wheel_link">
+    <link name="right_wheel">
         <visual>
             <origin xyz="0 0 0" rpy="${pi/2} 0 0"/>

File: src_ws/src/secbot_description/description/ros2_control.xacro (robot description, xacro)
@@ -72,9 +72,9 @@
     </xacro:if>
 -->
-<ros2_control name='RealRobot' type='system'>
+<ros2_control name="RealRobot" type="system">
             <hardware>
                 <plugin>diffdrive_arduino/DiffDriveArduinoHardware</plugin>
-                <param name="left_wheel_name">b_l_wheel_joint</param>
-                <param name="right_wheel_name">b_r_wheel_joint</param>
+                <param name="left_wheel_name">left_wheel_joint</param>
+                <param name="right_wheel_name">right_wheel_joint</param>
                 <param name="loop_rate">30</param>
                 <param name="device">/dev/ttyUSB1</param>
@@ -87,5 +87,5 @@
                 <param name="pid_o">50</param>
             </hardware>
-            <joint name="b_l_wheel_joint">
+            <joint name="left_wheel_joint">
                 <command_interface name="velocity">
                     <param name="min">-10</param>
@@ -95,5 +95,5 @@
                 <state_interface name="velocity" />
             </joint>
-            <joint name="b_r_wheel_joint">
+            <joint name="right_wheel_joint">
                 <command_interface name="velocity">
                     <param name="min">-10</param>

File: src_ws/src/secbot_description/description/sec_description.urdf.xacro (robot description, xacro)
@@ -2,5 +2,5 @@
 <robot name="sec_bot" xmlns:xacro="http://ros.org/wiki/xacro">
     <xacro:arg name="use_ros2_control" default="true"/>
-    <xacro:arg name="sim_mode" default="true"/>
+    <xacro:arg name="sim_mode" default="false"/>
     <xacro:property name="camera_x" value="0.010"/>
     <xacro:property name="camera_y" value="0.03"/>
