Commit message: updated urdf to accurately reflect wheel and chassis dimensions

File: src_ws/src/secbot_description/description/robot_core.xacro (robot description, xacro)
@@ -2,6 +2,4 @@
 <robot xmlns:xacro="http://ros.org/wiki/xacro">
     <xacro:include filename="inertial_macros.xacro"/>
-    <!-- The difference between bottom middle of chassis and wheel position(s)-->
-    <xacro:property name="wheel_x_displacement" value="0.08255"/>
     <!-- Base Link -->
     <link name="base_link"/>
@@ -18,5 +16,5 @@
         <parent link="base_link"/>
         <child link="chassis"/>
-        <origin xyz="0.0 0.0 ${chassis_z_offset}" rpy="0 0 0"/>
+        <origin xyz="0.0 0.0 ${wheel_radius/2 + chassis_z_offset}" rpy="0 0 0"/>
     </joint>
     <link name="chassis">
@@ -72,7 +70,7 @@
         </gazebo>
     </xacro:macro>
-    <xacro:wheel prefix="b_l" l_r="-1" f_b="1" />
-    <xacro:wheel prefix="b_r" l_r="-1" f_b="-1" />
-    <xacro:wheel prefix="f_l" l_r="1"  f_b="1" />
-    <xacro:wheel prefix="f_r" l_r="1"  f_b="-1" />
+    <xacro:wheel prefix="b_l" l_r="-1" f_b="-1" />
+    <xacro:wheel prefix="b_r" l_r="1" f_b="-1" />
+    <xacro:wheel prefix="f_l" l_r="-1"  f_b="1" />
+    <xacro:wheel prefix="f_r" l_r="1"  f_b="1" />
 </robot>

File: src_ws/src/secbot_description/description/robot_core_hw.xacro (robot description, xacro)
@@ -2,17 +2,6 @@
 <robot xmlns:xacro="http://ros.org/wiki/xacro">
     <xacro:include filename="inertial_macros.xacro"/>
-    <!-- Meters -->
-    <xacro:property name="chassis_length" value="0.205"/> <!--X-->
-    <xacro:property name="chassis_width" value="0.205"/> <!--Y-->
-    <xacro:property name="chassis_height" value="0.205"/> <!--Z-->
-    <xacro:property name="chassis_mass" value="10"/> <!--WHat is the unit for this?-->
-    <xacro:property name="chassis_z_offset" value="0.1"/> <!--Currently unused, going to try to implement for total height translation-->
-    <xacro:property name="wheel_radius" value="0.05"/> <!-- Update wheel radius paramter in controllers.yaml as well-->
-    <xacro:property name="wheel_length" value="0.025"/>
-    <xacro:property name="wheel_mass" value="10"/>
     <!-- The difference between bottom middle of chassis and wheel position(s)-->
     <xacro:property name="wheel_x_displacement" value="0.0"/>
-    <xacro:property name="wheel_y_displacement" value="0.115"/> <!-- Update wheel separation paramter in controllers.yaml as well-->
-    <xacro:property name="wheel_z_displacement" value="0.03"/>
     <!-- Base Link -->
     <link name="base_link"/>
@@ -29,5 +18,5 @@
         <parent link="base_link"/>
         <child link="chassis"/>
-        <origin xyz="0.0 0.0 ${wheel_radius/2 + chassis_z_offset}" rpy="0 0 0"/>
+        <origin xyz="0.0 0.0 ${chassis_z_offset}" rpy="0 0 0"/>
     </joint>
     <link name="chassis">

File: src_ws/src/secbot_description/description/sec_description.urdf.xacro (robot description, xacro)
@@ -12,4 +12,15 @@
     <xacro:property name="lidar_radius" value="0.05"/>
     <xacro:property name="lidar_length" value="0.04"/>
+    <!-- Meters -->
+    <xacro:property name="chassis_length" value="0.3048"/> <!--X-->
+    <xacro:property name="chassis_width" value="0.3048"/> <!--Y-->
+    <xacro:property name="chassis_height" value="0.2838"/> <!--Z-->
+    <xacro:property name="chassis_mass" value="10"/> <!--What is the unit for this?-->
+    <xacro:property name="chassis_z_offset" value="0.021"/> <!--Currently unused, going to try to implement for total height translation-->
+    <xacro:property name="wheel_radius" value="0.0381"/> <!-- Update wheel radius paramter in controllers.yaml as well-->
+    <xacro:property name="wheel_length" value="0.0254"/>
+    <xacro:property name="wheel_mass" value="10"/>
+    <xacro:property name="wheel_y_displacement" value="0.12065"/> <!-- Update wheel separation paramter in controllers.yaml as well-->
+    <xacro:property name="wheel_z_displacement" value="${wheel_radius/2}"/>
     <xacro:if value="$(arg sim_mode)">
         <xacro:include filename="robot_core_sim.xacro"/>
