Commit message: updated sensor urdf constants

File: src_ws/src/secbot_description/description/camera.xacro (robot description, xacro)
@@ -4,10 +4,10 @@
             <parent link="chassis"/>
             <child link="camera_link"/>
-            <origin xyz="${(chassis_length/2)+(camera_x/2)} 0 ${chassis_height/2}" rpy="0 0 0"/>
+            <origin xyz="${camera_x} ${camera_y} ${camera_z}" rpy="0 0 0"/>
         </joint>
         <link name="camera_link">
             <visual>
                 <geometry>
-                    <box size="${camera_x} ${camera_y} ${camera_z}"/>
+                    <box size="${camera_length} ${camera_width} ${camera_height}"/>
                 </geometry>
                 <material name="Gray">

File: src_ws/src/secbot_description/description/imu.xacro (robot description, xacro)
@@ -4,5 +4,5 @@
             <parent link="chassis"/>
             <child link="imu_link"/>
-            <origin xyz="-0.2 0 ${chassis_height+(imu_height/2)}" rpy="0 0 0"/>
+            <origin xyz="${imu_x} ${imu_y} ${imu_z}" rpy="0 0 0"/>
         </joint>
     <link name="imu_link">

File: src_ws/src/secbot_description/description/lidar.xacro (robot description, xacro)
@@ -4,5 +4,5 @@
             <parent link="chassis"/>
             <child link="lidar_link"/>
-            <origin xyz="0 0 ${chassis_height+(imu_height/2)}" rpy="0 0 0"/>
+            <origin xyz="${lidar_x} ${lidar_y} ${lidar_z}" rpy="0 0 0"/>
     </joint>
     <link name="lidar_link">

File: src_ws/src/secbot_description/description/sec_description.urdf.xacro (robot description, xacro)
@@ -3,13 +3,4 @@
     <xacro:arg name="use_ros2_control" default="true"/>
     <xacro:arg name="sim_mode" default="false"/>
-    <xacro:property name="camera_x" value="0.010"/>
-    <xacro:property name="camera_y" value="0.03"/>
-    <xacro:property name="camera_z" value="0.03"/>
-    <xacro:property name="camera_fov" value="1.089"/>
-    <xacro:property name="imu_length" value="0.05"/>
-    <xacro:property name="imu_width" value="0.05"/>
-    <xacro:property name="imu_height" value="0.02"/>
-    <xacro:property name="lidar_radius" value="0.05"/>
-    <xacro:property name="lidar_length" value="0.04"/>
     <!-- Meters -->
     <xacro:property name="chassis_length" value="0.3048"/> <!--X-->
@@ -23,4 +14,22 @@
     <xacro:property name="wheel_y_displacement" value="0.12065"/> <!-- Update wheel separation paramter in controllers.yaml as well-->
     <xacro:property name="wheel_z_displacement" value="${wheel_radius/2}"/>
+    <xacro:property name="camera_x" value="${-chassis_width/2}"/>
+    <xacro:property name="camera_y" value="0"/>
+    <xacro:property name="camera_z" value="${chassis_z_offset+chassis_height/2}"/>
+    <xacro:property name="camera_length" value="0.05"/>
+    <xacro:property name="camera_width" value="0.05"/>
+    <xacro:property name="camera_height" value="0.02"/>
+    <xacro:property name="camera_fov" value="1.089"/>
+    <xacro:property name="imu_x" value="0"/>
+    <xacro:property name="imu_y" value="0"/>
+    <xacro:property name="imu_z" value="${chassis_z_offset+chassis_height}"/>
+    <xacro:property name="imu_length" value="0.05"/>
+    <xacro:property name="imu_width" value="0.05"/>
+    <xacro:property name="imu_height" value="0.02"/>
+    <xacro:property name="lidar_x" value="${chassis_width/2}"/>
+    <xacro:property name="lidar_y" value="0"/>
+    <xacro:property name="lidar_z" value="${chassis_z_offset+chassis_height/2}"/>
+    <xacro:property name="lidar_radius" value="0.05"/>
+    <xacro:property name="lidar_length" value="0.04"/>
     <xacro:if value="$(arg sim_mode)">
         <xacro:include filename="robot_core_sim.xacro"/>
