Commit message: added system bringup launch file

File: src_ws/src/secbot_description/description/ros2_control.xacro (robot description, xacro)
@@ -6,35 +6,15 @@
                 <plugin><!-- PLACE MOTOR CONTROL PLUGIN HERE--></plugin>
             </hardware>
-            <joint name="b_l_wheel_joint">
-                <command_interface name="velocity">
-                    <param name="min">-10</param>
-                    <param name="max">10</param>
-                </command_interface>
-                <state_interface name="position" />
-                <state_interface name="velocity" />
+            <joint name="$l_wheel_joints" type="continuous">
+                <parent link="chassis"/>
+                <child link="${prefix}_wheel_link"/>
+                <origin xyz="${l_r*wheel_x_displacement} ${f_b*wheel_y_displacement} ${wheel_z_displacement}" rpy="0 0 0"/>
+                <axis xyz="0 1 0"/>
             </joint>
-            <joint name="b_r_wheel_joint">
-                <command_interface name="velocity">
-                    <param name="min">-10</param>
-                    <param name="max">10</param>
-                </command_interface>
-                <state_interface name="position" />
-                <state_interface name="velocity" />
-            </joint>
-            <joint name="f_l_wheel_joint">
-                <command_interface name="velocity">
-                    <param name="min">-10</param>
-                    <param name="max">10</param>
-                </command_interface>
-                <state_interface name="position" />
-                <state_interface name="velocity" />
-            </joint>
-            <joint name="f_r_wheel_joint">
-                <command_interface name="velocity">
-                    <param name="min">-10</param>
-                    <param name="max">10</param>
-                </command_interface>
-                <state_interface name="position" />
-                <state_interface name="velocity" />
+            <joint name="$r_wheel_joints" type="continuous">
+                <parent link="chassis"/>
+                <child link="${prefix}_wheel_link"/>
+                <origin xyz="${l_r*wheel_x_displacement} ${f_b*wheel_y_displacement} ${wheel_z_displacement}" rpy="0 0 0"/>
+                <axis xyz="0 1 0"/>
             </joint>
         </ros2_control>

Commit message: got software to run without removing hardware files, gonna try hw with steve now

File: src_ws/src/secbot_description/description/ros2_control.xacro (robot description, xacro)
@@ -1,33 +1,36 @@
 <?xml version="1.0"?>
 <robot xmlns:xacro="http://ros.org/wiki/xacro">
-<!--
     <xacro:unless value="$(arg sim_mode)">
         <ros2_control name="RealRobot" type="system">
             <hardware>
                 <plugin>diffdrive_arduino/DiffDriveArduinoHardware</plugin>
+                <param name="left_wheel_name">left_wheel_joint</param>
+                <param name="right_wheel_name">right_wheel_joint</param>
+                <param name="loop_rate">30</param>
+                <param name="device">/dev/ttyACM0</param>
+                <param name="baud_rate">57600</param>
+                <param name="timeout_ms">1000</param>
+                <param name="enc_counts_per_rev">3436</param>
+                <param name="pid_p">20</param>
+                <param name="pid_d">12</param>
+                <param name="pid_i">0</param>
+                <param name="pid_o">50</param>
             </hardware>
-            <joint name="l_wheel_joints" type="continuous">
-                <parent link="chassis"/>
-                <child link="l_wheel_link"/>
-                <origin xyz="${-1*wheel_x_displacement} ${0} ${wheel_z_displacement}" rpy="0 0 0"/>
-                <axis xyz="0 1 0"/>
+            <joint name="left_wheel_joint">
+                <command_interface name="velocity">
+                    <param name="min">-10</param>
+                    <param name="max">10</param>
+                </command_interface>
+                <state_interface name="position" />
+                <state_interface name="velocity" />
             </joint>
-            <joint name="r_wheel_joints" type="continuous">
-                <parent link="chassis"/>
-                <child link="r_wheel_link"/>
-                <origin xyz="${wheel_x_displacement} ${0} ${wheel_z_displacement}" rpy="0 0 0"/>
-                <axis xyz="0 1 0"/>
+            <joint name="right_wheel_joint">
+                <command_interface name="velocity">
+                    <param name="min">-10</param>
+                    <param name="max">10</param>
+                </command_interface>
+                <state_interface name="position" />
+                <state_interface name="velocity" />
             </joint>
-        </ros2_control>
-         IMU sensor-->
-        <!-- <ros2_control name='da_imu' type='sensor'>
-            <hardware>
-                <plugin>IMU SENSOR PLUGIN HERE</plugin>
-                <param name='sensor_name'>SAME AS IN controllers.yaml</param>
-                <param name='frame_id'>imu_link</param>
-            </hardware>
-            <sensor name=''>
-                STATE INTERFACES HERE
-            </sensor>
         </ros2_control>
     </xacro:unless>
@@ -70,61 +73,9 @@
             </joint>
         </ros2_control>
+        <gazebo>
+            <plugin filename="libgazebo_ros2_control.so" name="gazebo_ros2_control">
+                <parameters>$(find secbot_description)/config/controllers.yaml</parameters>
+            </plugin>
+        </gazebo>
     </xacro:if>
--->
-<ros2_control name="RealRobot" type="system">
-            <hardware>
-                <plugin>diffdrive_arduino/DiffDriveArduinoHardware</plugin>
-                <param name="left_wheel_name">left_wheel_joint</param>
-                <param name="right_wheel_name">right_wheel_joint</param>
-                <param name="loop_rate">30</param>
-                <param name="device">/dev/ttyACM0</param>
-                <param name="baud_rate">57600</param>
-                <param name="timeout_ms">1000</param>
-                <param name="enc_counts_per_rev">3436</param>
-                <param name="pid_p">20</param>
-                <param name="pid_d">12</param>
-                <param name="pid_i">0</param>
-                <param name="pid_o">50</param>
-            </hardware>
-            <joint name="left_wheel_joint">
-                <command_interface name="velocity">
-                    <param name="min">-10</param>
-                    <param name="max">10</param>
-                </command_interface>
-                <state_interface name="position" />
-                <state_interface name="velocity" />
-            </joint>
-            <joint name="right_wheel_joint">
-                <command_interface name="velocity">
-                    <param name="min">-10</param>
-                    <param name="max">10</param>
-                </command_interface>
-                <state_interface name="position" />
-                <state_interface name="velocity" />
-            </joint>
-<!--
-            <joint name="f_l_wheel_joint">
-                <command_interface name="velocity">
-                    <param name="min">-10</param>
-                    <param name="max">10</param>
-                </command_interface>
-                <state_interface name="position" />
-                <state_interface name="velocity" />
-            </joint>
-            <joint name="f_r_wheel_joint">
-                <command_interface name="velocity">
-                    <param name="min">-10</param>
-                    <param name="max">10</param>
-                </command_interface>
-                <state_interface name="position" />
-                <state_interface name="velocity" />
-            </joint>
--->
-        </ros2_control>
-<!--
-    <gazebo>
-        <plugin filename="libgazebo_ros2_control.so" name="gazebo_ros2_control">
-            <parameters>$(find secbot_description)/config/controllers.yaml</parameters>
-        </plugin>
-    </gazebo>-->
 </robot>
