Commit message: functional commit with first eleven waypoints and actions added, gonna tweak nav params

File: src_ws/src/secbot_description/description/sec_description.urdf.xacro (robot description, xacro)
@@ -29,5 +29,5 @@
     <xacro:property name="lidar_x" value="${chassis_width/2}"/>
     <xacro:property name="lidar_y" value="0"/>
-    <xacro:property name="lidar_z" value="${chassis_z_offset+chassis_height/2}"/>
+    <xacro:property name="lidar_z" value="${wheel_radius/2}"/>
     <xacro:property name="lidar_radius" value="0.05"/>
     <xacro:property name="lidar_length" value="0.04"/>
