Commit message: updated robot sim to only spawn two wheels on hardware bringup

File: src_ws/src/secbot_description/description/robot_core_sim.xacro (robot description, xacro)
@@ -2,4 +2,17 @@
 <robot xmlns:xacro="http://ros.org/wiki/xacro">
     <xacro:include filename="inertial_macros.xacro"/>
+    <!-- Meters -->
+    <xacro:property name="chassis_length" value="0.205"/> <!--X-->
+    <xacro:property name="chassis_width" value="0.205"/> <!--Y-->
+    <xacro:property name="chassis_height" value="0.205"/> <!--Z-->
+    <xacro:property name="chassis_mass" value="10"/> <!--WHat is the unit for this?-->
+    <xacro:property name="chassis_z_offset" value="0.1"/> <!--Currently unused, going to try to implement for total height translation-->
+    <xacro:property name="wheel_radius" value="0.05"/> <!-- Update wheel radius paramter in controllers.yaml as well-->
+    <xacro:property name="wheel_length" value="0.025"/>
+    <xacro:property name="wheel_mass" value="10"/>
+    <!-- The difference between bottom middle of chassis and wheel position(s)-->
+    <xacro:property name="wheel_x_displacement" value="${chassis_length/4}"/>
+    <xacro:property name="wheel_y_displacement" value="${chassis_width/2+wheel_radius}"/> <!-- Update wheel separation paramter in controllers.yaml as well-->
+    <xacro:property name="wheel_z_displacement" value="0.03"/>
     <!-- Base Link -->
     <link name="base_link"/>

File: src_ws/src/secbot_description/description/ros2_control.xacro (robot description, xacro)
@@ -40,14 +40,14 @@
         </ros2_control>
         <!-- IMU sensor-->
-        <ros2_control name='da_imu' type='sensor'>
+        <!-- <ros2_control name='da_imu' type='sensor'>
             <hardware>
-                <plugin><!--IMU SENSOR PLUGIN HERE--></plugin>
-                <param name='sensor_name'><!-- SAME AS IN controllers.yaml--></param>
+                <plugin>IMU SENSOR PLUGIN HERE</plugin>
+                <param name='sensor_name'>SAME AS IN controllers.yaml</param>
                 <param name='frame_id'>imu_link</param>
             </hardware>
             <sensor name=''>
-                <!--STATE INTERFACES HERE-->
+                STATE INTERFACES HERE
             </sensor>
-        </ros2_control>
+        </ros2_control>  -->
     </xacro:unless>
     <xacro:if value="$(arg sim_mode)">

File: src_ws/src/secbot_description/description/sec_description.urdf.xacro (robot description, xacro)
@@ -3,18 +3,4 @@
     <xacro:arg name="use_ros2_control" default="true"/>
     <xacro:arg name="sim_mode" default="true"/>
-    <!-- Define robot constants -->
-    <!-- Meters -->
-    <xacro:property name="chassis_length" value="0.205"/> <!--X-->
-    <xacro:property name="chassis_width" value="0.205"/> <!--Y-->
-    <xacro:property name="chassis_height" value="0.205"/> <!--Z-->
-    <xacro:property name="chassis_mass" value="10"/> <!--WHat is the unit for this?-->
-    <xacro:property name="chassis_z_offset" value="0.1"/> <!--Currently unused, going to try to implement for total height translation-->
-    <xacro:property name="wheel_radius" value="0.05"/> <!-- Update wheel radius paramter in controllers.yaml as well-->
-    <xacro:property name="wheel_length" value="0.025"/>
-    <xacro:property name="wheel_mass" value="10"/>
-    <!-- The difference between bottom middle of chassis and wheel position(s)-->
-    <xacro:property name="wheel_x_displacement" value="${chassis_length/4}"/>
-    <xacro:property name="wheel_y_displacement" value="${chassis_width/2+wheel_radius}"/> <!-- Update wheel separation paramter in controllers.yaml as well-->
-    <xacro:property name="wheel_z_displacement" value="0.03"/>
     <xacro:property name="camera_x" value="0.010"/>
     <xacro:property name="camera_y" value="0.03"/>
@@ -26,8 +12,13 @@
     <xacro:property name="lidar_radius" value="0.05"/>
     <xacro:property name="lidar_length" value="0.04"/>
-    <xacro:include filename="robot_core.xacro"/>
     <xacro:include filename="camera.xacro"/>
     <xacro:include filename="imu.xacro"/>
     <xacro:include filename="lidar.xacro"/>
+    <xacro:if value="$(arg sim_mode)">
+        <xacro:include filename="robot_core_sim.xacro"/>
+    </xacro:if>
+    <xacro:unless value="$(arg sim_mode)">
+        <xacro:include filename="robot_core_hw.xacro" />
+    </xacro:unless>
     <xacro:if value="$(arg use_ros2_control)">
         <xacro:include filename="ros2_control.xacro" />

Commit message: changed robot size, made new comp course and map, redid every waypoint, and tweaked nav2_params params

File: src_ws/src/secbot_description/description/robot_core_sim.xacro (robot description, xacro)
@@ -3,5 +3,5 @@
     <xacro:include filename="inertial_macros.xacro"/>
     <!-- The difference between bottom middle of chassis and wheel position(s)-->
-    <xacro:property name="wheel_x_displacement" value="0.08255"/>
+    <xacro:property name="wheel_x_displacement" value="0.09255"/>
     <!-- Base Link -->
     <link name="base_link"/>
