Commit message: made gazebo use og comp course, changed up urdf, made new comp course map, and changed some waypoint implementation

File: src_ws/src/secbot_description/description/lidar.xacro (robot description, xacro)
@@ -4,5 +4,5 @@
             <parent link="chassis"/>
             <child link="lidar_link"/>
-            <origin xyz="0 0 ${chassis_height+(imu_height/2)}" rpy="0 0 0"/>
+            <origin xyz="0.09 0 .025" rpy="0 0 0"/>
     </joint>
     <link name="lidar_link">

File: src_ws/src/secbot_description/description/robot_core_sim.xacro (robot description, xacro)
@@ -12,6 +12,6 @@
     <xacro:property name="wheel_mass" value="10"/>
     <!-- The difference between bottom middle of chassis and wheel position(s)-->
-    <xacro:property name="wheel_x_displacement" value="${chassis_length/4}"/>
-    <xacro:property name="wheel_y_displacement" value="${chassis_width/2+wheel_radius}"/> <!-- Update wheel separation paramter in controllers.yaml as well-->
+    <xacro:property name="wheel_x_displacement" value="${chassis_length/3}"/>
+    <xacro:property name="wheel_y_displacement" value="${chassis_width/2+wheel_length}"/> <!-- Update wheel separation paramter in controllers.yaml as well-->
     <xacro:property name="wheel_z_displacement" value="0.03"/>
     <!-- Base Link -->

Commit message: fixed controllers.yaml configs and made entire the sim use a flat course

File: src_ws/src/secbot_description/description/lidar.xacro (robot description, xacro)
@@ -30,6 +30,6 @@
                     <samples>360</samples>
                     <resolution>1</resolution>
-                    <min_angle>-1.57</min_angle>
-                    <max_angle>1.57</max_angle>
+                    <min_angle>-3.14</min_angle>
+                    <max_angle>3.14</max_angle>
                     </horizontal>
                 </scan>

File: src_ws/src/secbot_description/description/sec_description.urdf.xacro (robot description, xacro)
@@ -14,5 +14,5 @@
     <xacro:property name="wheel_y_displacement" value="0.12065"/> <!-- Update wheel separation paramter in controllers.yaml as well-->
     <xacro:property name="wheel_z_displacement" value="${wheel_radius/2}"/>
-    <xacro:property name="camera_x" value="${-chassis_width/2}"/>
+    <xacro:property name="camera_x" value="${chassis_width/2}"/>
     <xacro:property name="camera_y" value="0"/>
     <xacro:property name="camera_z" value="${chassis_z_offset+chassis_height/2}"/>
@@ -27,7 +27,7 @@
     <xacro:property name="imu_width" value="0.05"/>
     <xacro:property name="imu_height" value="0.02"/>
-    <xacro:property name="lidar_x" value="${chassis_width/2}"/>
+    <xacro:property name="lidar_x" value="0"/>
     <xacro:property name="lidar_y" value="0"/>
-    <xacro:property name="lidar_z" value="${wheel_radius/2}"/>
+    <xacro:property name="lidar_z" value="${chassis_height+lidar_length/2}"/>
     <xacro:property name="lidar_radius" value="0.05"/>
     <xacro:property name="lidar_length" value="0.04"/>
